Commit message: 3 link, 2 joint

File: body.urdf (robot description, URDF)
Before this commit: robot robot, 7 links, 6 joints
Links:
- removed link Link0
- removed link Link1
- removed link Link2
- removed link Link3
- removed link Link4
- removed link Link5
- removed link Link6
- added link BackLeg, mass 1; collision box size=1 1 1; visual box size=1 1 1
- added link FrontLeg, mass 1; collision box size=1 1 1; visual box size=1 1 1
- added link Torso, mass 1; collision box size=1 1 1; visual box size=1 1 1
Joints:
- removed joint Link0_Link1
- removed joint Link1_Link2
- removed joint Link2_Link3
- removed joint Link3_Link4
- removed joint Link4_Link5
- removed joint Link5_Link6
- added joint Torso_BackLeg: type revolute, parent Torso, child BackLeg, origin xyz=1 0 1 rpy=0 0 0, axis 0 1 0, limit lower=-3.14159 upper=3.14159 effort=0.0 velocity=0.0
- added joint Torso_FrontLeg: type revolute, parent Torso, child FrontLeg, origin xyz=2 0 1 rpy=0 0 0, axis 0 1 0, limit lower=-3.14159 upper=3.14159 effort=0.0 velocity=0.0

Commit message: try

File: body.urdf (robot description, URDF)
Before this commit: robot robot, 9 links, 8 joints
Links:
- removed link BackLeg
- removed link BackLowerLeg
- removed link FrontLeg
- removed link FrontLowerLeg
- removed link LeftLeg
- removed link LeftLowerLeg
- removed link RightLeg
- removed link RightLowerLeg
- added link LeftLeg1, mass 1; collision box size=0.2 1 0.2; visual box size=0.2 1 0.2
- added link LeftLeg2, mass 1; collision box size=0.2 1 0.2; visual box size=0.2 1 0.2
- added link LeftLeg3, mass 1; collision box size=0.2 1 0.2; visual box size=0.2 1 0.2
- added link LeftLowerLeg1, mass 1; collision box size=0.2 0.2 1; visual box size=0.2 0.2 1
- added link LeftLowerLeg2, mass 1; collision box size=0.2 0.2 1; visual box size=0.2 0.2 1
- added link LeftLowerLeg3, mass 1; collision box size=0.2 0.2 1; visual box size=0.2 0.2 1
- added link RightLeg1, mass 1; collision box size=0.2 1 0.2; visual box size=0.2 1 0.2
- added link RightLeg2, mass 1; collision box size=0.2 1 0.2; visual box size=0.2 1 0.2
- added link RightLeg3, mass 1; collision box size=0.2 1 0.2; visual box size=0.2 1 0.2
- added link RightLowerLeg1, mass 1; collision box size=0.2 0.2 1; visual box size=0.2 0.2 1
- added link RightLowerLeg2, mass 1; collision box size=0.2 0.2 1; visual box size=0.2 0.2 1
- added link RightLowerLeg3, mass 1; collision box size=0.2 0.2 1; visual box size=0.2 0.2 1
- added link Tail, mass 1; collision box size=2 0.4 0.2; visual box size=2 0.4 0.2
- link Torso: geometry collision box size=3 1 1; visual box size=3 1 1
Joints:
- removed joint BackLeg_BackLowerLeg
- removed joint FrontLeg_FrontLowerLeg
- removed joint LeftLeg_LeftLowerLeg
- removed joint RightLeg_RightLowerLeg
- removed joint Torso_BackLeg
- removed joint Torso_FrontLeg
- removed joint Torso_LeftLeg
- removed joint Torso_RightLeg
- added joint LeftLeg1_LeftLowerLeg1: type revolute, parent LeftLeg1, child LeftLowerLeg1, origin xyz=0 -1 0 rpy=0 0 0, axis 1 0 0, limit lower=-3.14159 upper=3.14159 effort=0.0 velocity=0.0
- added joint LeftLeg2_LeftLowerLeg2: type revolute, parent LeftLeg2, child LeftLowerLeg2, origin xyz=0 -1 0 rpy=0 0 0, axis 1 0 0, limit lower=-3.14159 upper=3.14159 effort=0.0 velocity=0.0
- added joint LeftLeg3_LeftLowerLeg3: type revolute, parent LeftLeg3, child LeftLowerLeg3, origin xyz=0 -1 0 rpy=0 0 0, axis 1 0 0, limit lower=-3.14159 upper=3.14159 effort=0.0 velocity=0.0
- added joint RightLeg1_RightLowerLeg1: type revolute, parent RightLeg1, child RightLowerLeg1, origin xyz=0 1 0 rpy=0 0 0, axis 1 0 0, limit lower=-3.14159 upper=3.14159 effort=0.0 velocity=0.0
- added joint RightLeg2_RightLowerLeg2: type revolute, parent RightLeg2, child RightLowerLeg2, origin xyz=0 1 0 rpy=0 0 0, axis 1 0 0, limit lower=-3.14159 upper=3.14159 effort=0.0 velocity=0.0
- added joint RightLeg3_RightLowerLeg3: type revolute, parent RightLeg3, child RightLowerLeg3, origin xyz=0 1 0 rpy=0 0 0, axis 1 0 0, limit lower=-3.14159 upper=3.14159 effort=0.0 velocity=0.0
- added joint Torso_LeftLeg1: type revolute, parent Torso, child LeftLeg1, origin xyz=-1 -0.5 3 rpy=0 0 0, axis 1 0 0, limit lower=-3.14159 upper=3.14159 effort=0.0 velocity=0.0
- added joint Torso_LeftLeg2: type revolute, parent Torso, child LeftLeg2, origin xyz=0 -0.5 3 rpy=0 0 0, axis 1 0 0, limit lower=-3.14159 upper=3.14159 effort=0.0 velocity=0.0
- added joint Torso_LeftLeg3: type revolute, parent Torso, child LeftLeg3, origin xyz=1 -0.5 3 rpy=0 0 0, axis 1 0 0, limit lower=-3.14159 upper=3.14159 effort=0.0 velocity=0.0
- added joint Torso_RightLeg1: type revolute, parent Torso, child RightLeg1, origin xyz=-1 0.5 3 rpy=0 0 0, axis 1 0 0, limit lower=-3.14159 upper=3.14159 effort=0.0 velocity=0.0
- added joint Torso_RightLeg2: type revolute, parent Torso, child RightLeg2, origin xyz=0 0.5 3 rpy=0 0 0, axis 1 0 0, limit lower=-3.14159 upper=3.14159 effort=0.0 velocity=0.0
- added joint Torso_RightLeg3: type revolute, parent Torso, child RightLeg3, origin xyz=1 0.5 3 rpy=0 0 0, axis 1 0 0, limit lower=-3.14159 upper=3.14159 effort=0.0 velocity=0.0
- added joint Torso_Tail: type revolute, parent Torso, child Tail, origin xyz=1 0 3 rpy=0 0 0, axis 0 1 0, limit lower=-3.14159 upper=3.14159 effort=0.0 velocity=0.0

Commit message: Finished Bot

File: body.urdf (robot description, URDF)
Before this commit: robot robot, 14 links, 13 joints
Links:
- removed link LeftLeg1
- removed link LeftLeg2
- removed link LeftLeg3
- removed link LeftLowerLeg1
- removed link LeftLowerLeg2
- removed link LeftLowerLeg3
- removed link RightLeg1
- removed link RightLeg2
- removed link RightLeg3
- removed link RightLowerLeg1
- removed link RightLowerLeg2
- removed link RightLowerLeg3
- removed link Tail
- added link Butt, mass 1; collision box size=1 0.2 0.2; visual box size=1 0.2 0.2
- added link Head, mass 1; collision box size=1 0.2 0.2; visual box size=1 0.2 0.2
- link Torso: geometry collision box size=1 0.2 0.2; visual box size=1 0.2 0.2
Joints:
- removed joint LeftLeg1_LeftLowerLeg1
- removed joint LeftLeg2_LeftLowerLeg2
- removed joint LeftLeg3_LeftLowerLeg3
- removed joint RightLeg1_RightLowerLeg1
- removed joint RightLeg2_RightLowerLeg2
- removed joint RightLeg3_RightLowerLeg3
- removed joint Torso_LeftLeg1
- removed joint Torso_LeftLeg2
- removed joint Torso_LeftLeg3
- removed joint Torso_RightLeg1
- removed joint Torso_RightLeg2
- removed joint Torso_RightLeg3
- removed joint Torso_Tail
- added joint Torso_Butt: type revolute, parent Torso, child Butt, origin xyz=0.5 0 0 rpy=0 0 0, axis 0 1 0, limit lower=-3.14159 upper=3.14159 effort=0.0 velocity=0.0
- added joint Torso_Head: type revolute, parent Torso, child Head, origin xyz=-0.5 0 0 rpy=0 0 0, axis 1 0 0, limit lower=-3.14159 upper=3.14159 effort=0.0 velocity=0.0

Commit message: sad attempt

File: body.urdf (robot description, URDF)
Before this commit: robot robot, 3 links, 2 joints
Links:
- removed link Butt
- removed link Head
- added link Link0, mass 1; collision box size=2.721834633699328 0.2 0.2; visual box size=2.721834633699328 0.2 0.2
- added link Link1, mass 1; collision box size=3.982158179485533 0.2 0.2; visual box size=3.982158179485533 0.2 0.2
- added link Link2, mass 1; collision box size=3.753828258972509 0.2 0.2; visual box size=3.753828258972509 0.2 0.2
- added link Link3, mass 1; collision box size=0.20028390185504508 0.2 0.2; visual box size=0.20028390185504508 0.2 0.2
- added link Link4, mass 1; collision box size=9.779439208445401 0.2 0.2; visual box size=9.779439208445401 0.2 0.2
- added link Link5, mass 1; collision box size=9.507862270663598 0.2 0.2; visual box size=9.507862270663598 0.2 0.2
- added link Link6, mass 1; collision box size=2.6960946904232594 0.2 0.2; visual box size=2.6960946904232594 0.2 0.2
Joints:
- removed joint Torso_Butt
- removed joint Torso_Head
- added joint Joint0: type revolute, parent Torso, child Link0, origin xyz=0.5 0 0 rpy=0 0 0, axis 0 1 0, limit lower=-3.14159 upper=3.14159 effort=0.0 velocity=0.0
- added joint Joint1: type revolute, parent Link0, child Link1, origin xyz=3.982158179485533 0 0 rpy=0 0 0, axis 0 1 0, limit lower=-3.14159 upper=3.14159 effort=0.0 velocity=0.0
- added joint Joint2: type revolute, parent Link1, child Link2, origin xyz=3.753828258972509 0 0 rpy=0 0 0, axis 0 1 0, limit lower=-3.14159 upper=3.14159 effort=0.0 velocity=0.0
- added joint Joint3: type revolute, parent Link2, child Link3, origin xyz=0.20028390185504508 0 0 rpy=0 0 0, axis 0 1 0, limit lower=-3.14159 upper=3.14159 effort=0.0 velocity=0.0
- added joint Joint4: type revolute, parent Link3, child Link4, origin xyz=9.779439208445401 0 0 rpy=0 0 0, axis 0 1 0, limit lower=-3.14159 upper=3.14159 effort=0.0 velocity=0.0
- added joint Joint5: type revolute, parent Link4, child Link5, origin xyz=9.507862270663598 0 0 rpy=0 0 0, axis 0 1 0, limit lower=-3.14159 upper=3.14159 effort=0.0 velocity=0.0
- added joint Joint6: type revolute, parent Link5, child Link6, origin xyz=2.6960946904232594 0 0 rpy=0 0 0, axis 0 1 0, limit lower=-3.14159 upper=3.14159 effort=0.0 velocity=0.0

Commit message: Finished Random Snakes w Color

File: body.urdf (robot description, URDF)
Before this commit: robot robot, 3 links, 2 joints
Links:
- removed link Butt
- removed link Head
- removed link Torso
- added link Link0, mass 1; collision box size=3.8918515877238207 3.167738937934442 0.6230494825574655; visual box size=3.8918515877238207 3.167738937934442 0.6230494825574655
- added link Link1, mass 1; collision box size=3.5930932313496227 2.308784615691909 3.0763442463966046; visual box size=3.5930932313496227 2.308784615691909 3.0763442463966046
- added link Link10, mass 1; collision box size=2.640345151800351 0.23046516861297617 0.05999331319782364; visual box size=2.640345151800351 0.23046516861297617 0.05999331319782364
- added link Link11, mass 1; collision box size=1.6407092614361325 1.1574422734727103 2.887586032417801; visual box size=1.6407092614361325 1.1574422734727103 2.887586032417801
- added link Link12, mass 1; collision box size=3.2906785199519146 2.17200202936229 2.9867876195666927; visual box size=3.2906785199519146 2.17200202936229 2.9867876195666927
- added link Link13, mass 1; collision box size=3.2556396055350825 3.361260639144413 3.609137953898541; visual box size=3.2556396055350825 3.361260639144413 3.609137953898541
- added link Link14, mass 1; collision box size=2.714930351847133 3.302773329075415 1.1425150906666852; visual box size=2.714930351847133 3.302773329075415 1.1425150906666852
- added link Link15, mass 1; collision box size=2.2494762989844035 3.1176547460466386 3.9856163660675437; visual box size=2.2494762989844035 3.1176547460466386 3.9856163660675437
- added link Link16, mass 1; collision box size=0.5377426406627417 0.4509859730226786 2.202625081817556; visual box size=0.5377426406627417 0.4509859730226786 2.202625081817556
- added link Link2, mass 1; collision box size=3.6448790306063312 2.677172982005047 1.4472761129345684; visual box size=3.6448790306063312 2.677172982005047 1.4472761129345684
- added link Link3, mass 1; collision box size=0.6168422447544146 3.4798092708117134 1.912458998067995; visual box size=0.6168422447544146 3.4798092708117134 1.912458998067995
- added link Link4, mass 1; collision box size=2.5726819376764296 3.251005758261793 1.8855247520831067; visual box size=2.5726819376764296 3.251005758261793 1.8855247520831067
- added link Link5, mass 1; collision box size=1.4098862465024138 0.5346179744181545 3.0511286130316333; visual box size=1.4098862465024138 0.5346179744181545 3.0511286130316333
- added link Link6, mass 1; collision box size=3.3101291704539606 2.8946142642090793 3.6594831514126187; visual box size=3.3101291704539606 2.8946142642090793 3.6594831514126187
- added link Link7, mass 1; collision box size=1.894111273888901 3.6011591822214304 0.35741582500801083; visual box size=1.894111273888901 3.6011591822214304 0.35741582500801083
- added link Link8, mass 1; collision box size=0.4579915645837511 3.9633060926406447 1.2250919841197772; visual box size=0.4579915645837511 3.9633060926406447 1.2250919841197772
- added link Link9, mass 1; collision box size=2.483065452816089 3.1032743837181873 1.0188512419612534; visual box size=2.483065452816089 3.1032743837181873 1.0188512419612534
Joints:
- removed joint Torso_Butt
- removed joint Torso_Head
- added joint Link0_Link1: type revolute, parent Link0, child Link1, origin xyz=3.8918515877238207 0 5 rpy=0 0 0, axis 0 0 1, limit lower=-3.14159 upper=3.14159 effort=0.0 velocity=0.0
- added joint Link10_Link11: type revolute, parent Link10, child Link11, origin xyz=2.640345151800351 0 0 rpy=0 0 0, axis 0 0 1, limit lower=-3.14159 upper=3.14159 effort=0.0 velocity=0.0
- added joint Link11_Link12: type revolute, parent Link11, child Link12, origin xyz=1.6407092614361325 0 0 rpy=0 0 0, axis 0 0 1, limit lower=-3.14159 upper=3.14159 effort=0.0 velocity=0.0
- added joint Link12_Link13: type revolute, parent Link12, child Link13, origin xyz=3.2906785199519146 0 0 rpy=0 0 0, axis 0 0 1, limit lower=-3.14159 upper=3.14159 effort=0.0 velocity=0.0
- added joint Link13_Link14: type revolute, parent Link13, child Link14, origin xyz=3.2556396055350825 0 0 rpy=0 0 0, axis 0 0 1, limit lower=-3.14159 upper=3.14159 effort=0.0 velocity=0.0
- added joint Link14_Link15: type revolute, parent Link14, child Link15, origin xyz=2.714930351847133 0 0 rpy=0 0 0, axis 0 0 1, limit lower=-3.14159 upper=3.14159 effort=0.0 velocity=0.0
- added joint Link15_Link16: type revolute, parent Link15, child Link16, origin xyz=2.2494762989844035 0 0 rpy=0 0 0, axis 0 0 1, limit lower=-3.14159 upper=3.14159 effort=0.0 velocity=0.0
- added joint Link1_Link2: type revolute, parent Link1, child Link2, origin xyz=3.5930932313496227 0 0 rpy=0 0 0, axis 0 0 1, limit lower=-3.14159 upper=3.14159 effort=0.0 velocity=0.0
- added joint Link2_Link3: type revolute, parent Link2, child Link3, origin xyz=3.6448790306063312 0 0 rpy=0 0 0, axis 0 0 1, limit lower=-3.14159 upper=3.14159 effort=0.0 velocity=0.0
- added joint Link3_Link4: type revolute, parent Link3, child Link4, origin xyz=0.6168422447544146 0 0 rpy=0 0 0, axis 0 0 1, limit lower=-3.14159 upper=3.14159 effort=0.0 velocity=0.0
- added joint Link4_Link5: type revolute, parent Link4, child Link5, origin xyz=2.5726819376764296 0 0 rpy=0 0 0, axis 0 0 1, limit lower=-3.14159 upper=3.14159 effort=0.0 velocity=0.0
- added joint Link5_Link6: type revolute, parent Link5, child Link6, origin xyz=1.4098862465024138 0 0 rpy=0 0 0, axis 0 0 1, limit lower=-3.14159 upper=3.14159 effort=0.0 velocity=0.0
- added joint Link6_Link7: type revolute, parent Link6, child Link7, origin xyz=3.3101291704539606 0 0 rpy=0 0 0, axis 0 0 1, limit lower=-3.14159 upper=3.14159 effort=0.0 velocity=0.0
- added joint Link7_Link8: type revolute, parent Link7, child Link8, origin xyz=1.894111273888901 0 0 rpy=0 0 0, axis 0 0 1, limit lower=-3.14159 upper=3.14159 effort=0.0 velocity=0.0
- added joint Link8_Link9: type revolute, parent Link8, child Link9, origin xyz=0.4579915645837511 0 0 rpy=0 0 0, axis 0 0 1, limit lower=-3.14159 upper=3.14159 effort=0.0 velocity=0.0
- added joint Link9_Link10: type revolute, parent Link9, child Link10, origin xyz=2.483065452816089 0 0 rpy=0 0 0, axis 0 0 1, limit lower=-3.14159 upper=3.14159 effort=0.0 velocity=0.0

Commit message: 3D Plane Random Creature Generation
Successfully sends links and joints. Not connected though. Need to fix

File: body.urdf (robot description, URDF)
Before this commit: robot robot, 17 links, 16 joints
Links:
- removed link Link10
- removed link Link11
- removed link Link12
- removed link Link13
- removed link Link14
- removed link Link15
- removed link Link16
- removed link Link5
- removed link Link6
- removed link Link7
- removed link Link8
- removed link Link9
- link Link0: geometry collision box size=1.244571280113945 1.6246838587290648 0.4431488117359117; visual box size=1.244571280113945 1.6246838587290648 0.4431488117359117
- link Link1: geometry collision box size=1.877569484113447 0.9774425022666531 2.9296025343066554; visual box size=1.877569484113447 0.9774425022666531 2.9296025343066554
- link Link2: geometry collision box size=1.8493993521311722 2.9704815589149063 1.1352182499354004; visual box size=1.8493993521311722 2.9704815589149063 1.1352182499354004
- link Link3: geometry collision box size=2.320314814156936 1.2409562227932045 0.9029427290187421; visual box size=2.320314814156936 1.2409562227932045 0.9029427290187421
- link Link4: geometry collision box size=0.048077518620780135 2.350851471711956 0.11761415139288056; visual box size=0.048077518620780135 2.350851471711956 0.11761415139288056
Joints:
- removed joint Link10_Link11
- removed joint Link11_Link12
- removed joint Link12_Link13
- removed joint Link13_Link14
- removed joint Link14_Link15
- removed joint Link15_Link16
- removed joint Link1_Link2
- removed joint Link2_Link3
- removed joint Link3_Link4
- removed joint Link4_Link5
- removed joint Link5_Link6
- removed joint Link6_Link7
- removed joint Link7_Link8
- removed joint Link8_Link9
- removed joint Link9_Link10
- added joint Link0_Link2: type revolute, parent Link0, child Link2, origin xyz=0 2.9704815589149063 0 rpy=0 0 0, axis 0 0 1, limit lower=-3.14159 upper=3.14159 effort=0.0 velocity=0.0
- added joint Link1_Link3: type revolute, parent Link1, child Link3, origin xyz=-2.320314814156936 0 0 rpy=0 0 0, axis 0 1 0, limit lower=-3.14159 upper=3.14159 effort=0.0 velocity=0.0
- added joint Link2_Link4: type revolute, parent Link2, child Link4, origin xyz=-0.048077518620780135 0 0 rpy=0 0 0, axis 0 0 1, limit lower=-3.14159 upper=3.14159 effort=0.0 velocity=0.0
- joint Link0_Link1: origin xyz=3.8918515877238207 0 5 rpy=0 0 0 -> xyz=-1.877569484113447 0 0 rpy=0 0 0

Commit message: Fixed Joints

File: body.urdf (robot description, URDF)
Before this commit: robot robot, 5 links, 4 joints
Links:
- added link Link5, mass 1; collision box size=2.3929821381553658 1.8091875362799787 0.9489908830257302; visual box size=2.3929821381553658 1.8091875362799787 0.9489908830257302
- added link Link6, mass 1; collision box size=1.7871701322092117 2.4398499561426736 0.13110152482520165; visual box size=1.7871701322092117 2.4398499561426736 0.13110152482520165
- link Link0: geometry collision box size=1.778530459355741 2.149331666034851 2.530180172316633; visual box size=1.778530459355741 2.149331666034851 2.530180172316633
- link Link1: geometry collision box size=2.519402392354692 1.0443800706951571 1.4514876742175322; visual box size=2.519402392354692 1.0443800706951571 1.4514876742175322
- link Link2: geometry collision box size=2.264819362510715 0.046390131450309124 0.07520258293323867; visual box size=2.264819362510715 0.046390131450309124 0.07520258293323867
- link Link3: geometry collision box size=0.8953379720589855 2.9800559929471953 0.877554645437496; visual box size=0.8953379720589855 2.9800559929471953 0.877554645437496
- link Link4: geometry collision box size=1.6138357219445132 2.149576930192999 1.1868876319218682; visual box size=1.6138357219445132 2.149576930192999 1.1868876319218682
Joints:
- removed joint Link0_Link2
- removed joint Link1_Link3
- removed joint Link2_Link4
- added joint Link1_Link2: type revolute, parent Link1, child Link2, origin xyz=0 -0.5221900353475786 0.7257438371087661 rpy=0 0 0, axis 1 0 0, limit lower=-3.14159 upper=3.14159 effort=0.0 velocity=0.0
- added joint Link1_Link5: type revolute, parent Link1, child Link5, origin xyz=-1.259701196177346 0 0.7257438371087661 rpy=0 0 0, axis 0 1 0, limit lower=-3.14159 upper=3.14159 effort=0.0 velocity=0.0
- added joint Link1_Link6: type revolute, parent Link1, child Link6, origin xyz=1.259701196177346 0 0.7257438371087661 rpy=0 0 0, axis 0 1 0, limit lower=-3.14159 upper=3.14159 effort=0.0 velocity=0.0
- added joint Link2_Link3: type revolute, parent Link2, child Link3, origin xyz=0 -0.023195065725154562 -0.037601291466619335 rpy=0 0 0, axis 0 1 0, limit lower=-3.14159 upper=3.14159 effort=0.0 velocity=0.0
- added joint Link3_Link4: type revolute, parent Link3, child Link4, origin xyz=0 0 -0.877554645437496 rpy=0 0 0, axis 1 0 0, limit lower=-3.14159 upper=3.14159 effort=0.0 velocity=0.0
- joint Link0_Link1: axis 0 0 1 -> 0 1 0; origin xyz=-1.877569484113447 0 0 rpy=0 0 0 -> xyz=0 0 4.265090086158317 rpy=0 0 0
