Commit message: Finished!

File: body.urdf (robot description, URDF)
Before this commit: robot robot, 7 links, 6 joints
Links:
- added link Link7, mass 1; collision box size=2.603578401840637 0.6297028389797509 2.442849824599411; visual box size=2.603578401840637 0.6297028389797509 2.442849824599411
- added link Link8, mass 1; collision box size=2.5173041990042813 0.0501682333537683 0.8049969244620753; visual box size=2.5173041990042813 0.0501682333537683 0.8049969244620753
- added link Link9, mass 1; collision box size=1.5040200914848176 2.7899271427925183 0.21867800717116614; visual box size=1.5040200914848176 2.7899271427925183 0.21867800717116614
- link Link0: geometry collision box size=2.847263001743226 0.6827580057286418 1.0358175674747148; visual box size=2.847263001743226 0.6827580057286418 1.0358175674747148
- link Link1: geometry collision box size=1.280881911654471 0.7396185975921371 0.010280393360587503; visual box size=1.280881911654471 0.7396185975921371 0.010280393360587503
- link Link2: geometry collision box size=1.4291170016434753 1.7311410195092565 1.972219973478575; visual box size=1.4291170016434753 1.7311410195092565 1.972219973478575
- link Link3: geometry collision box size=1.8029834251498742 1.0650020408102128 2.2899967753527726; visual box size=1.8029834251498742 1.0650020408102128 2.2899967753527726
- link Link4: geometry collision box size=1.7968411972200926 1.3804440121793449 2.7045312183318693; visual box size=1.7968411972200926 1.3804440121793449 2.7045312183318693
- link Link5: geometry collision box size=1.2775042189948027 2.7736498572991315 0.7723474154629655; visual box size=1.2775042189948027 2.7736498572991315 0.7723474154629655
- link Link6: geometry collision box size=2.0547782695333012 2.7547224396791106 1.5640903341009678; visual box size=2.0547782695333012 2.7547224396791106 1.5640903341009678
Joints:
- removed joint Link1_Link5
- removed joint Link1_Link6
- removed joint Link3_Link4
- added joint Link0_Link7: type revolute, parent Link0, child Link7, origin xyz=0 0.3413790028643209 3 rpy=0 0 0, axis 0 0 1, limit lower=-3.14159 upper=3.14159 effort=0.0 velocity=0.0
- added joint Link2_Link4: type revolute, parent Link2, child Link4, origin xyz=0 -1.7311410195092565 0 rpy=0 0 0, axis 1 0 0, limit lower=-3.14159 upper=3.14159 effort=0.0 velocity=0.0
- added joint Link3_Link5: type revolute, parent Link3, child Link5, origin xyz=-0.9014917125749371 -0.5325010204051064 0 rpy=0 0 0, axis 1 0 0, limit lower=-3.14159 upper=3.14159 effort=0.0 velocity=0.0
- added joint Link3_Link6: type revolute, parent Link3, child Link6, origin xyz=-0.9014917125749371 0 1.1449983876763863 rpy=0 0 0, axis 1 0 0, limit lower=-3.14159 upper=3.14159 effort=0.0 velocity=0.0
- added joint Link4_Link9: type revolute, parent Link4, child Link9, origin xyz=0.8984205986100463 -0.6902220060896724 0 rpy=0 0 0, axis 1 0 0, limit lower=-3.14159 upper=3.14159 effort=0.0 velocity=0.0
- added joint Link7_Link8: type revolute, parent Link7, child Link8, origin xyz=0 0.31485141948987544 1.2214249122997054 rpy=0 0 0, axis 0 1 0, limit lower=-3.14159 upper=3.14159 effort=0.0 velocity=0.0
- joint Link0_Link1: axis 0 1 0 -> 0 0 1; origin xyz=0 0 4.265090086158317 rpy=0 0 0 -> xyz=-1.423631500871613 0 3 rpy=0 0 0
- joint Link1_Link2: axis 1 0 0 -> 0 1 0; origin xyz=0 -0.5221900353475786 0.7257438371087661 rpy=0 0 0 -> xyz=-0.6404409558272355 -0.36980929879606855 0 rpy=0 0 0
- joint Link2_Link3: axis 0 1 0 -> 0 0 1; origin xyz=0 -0.023195065725154562 -0.037601291466619335 rpy=0 0 0 -> xyz=-0.7145585008217377 -0.8655705097546282 0 rpy=0 0 0
