Commit message: Samples 0 - 4

File: samples/sample_2/body2a.urdf (robot description, URDF)
Before this commit: robot robot, 4 links, 3 joints
Links:
- removed link Link4
- added link Link2, mass 1; collision box size=0.7738494630704211 1.4638116451055658 0.059993078090504304; visual box size=0.7738494630704211 1.4638116451055658 0.059993078090504304
- link Link0: geometry collision box size=0.019308650023105167 0.04254870048121806 1.2615485263121426; visual box size=0.019308650023105167 0.04254870048121806 1.2615485263121426
- link Link1: geometry collision box size=1.0953976153862566 1.0521638401589435 1.3797442974900953; visual box size=1.0953976153862566 1.0521638401589435 1.3797442974900953
- link Link3: geometry collision box size=0.008810241711453115 1.3701065836090018 0.4138378074451731; visual box size=0.008810241711453115 1.3701065836090018 0.4138378074451731
Joints:
- removed joint Link0_Link4
- added joint Link0_Link2: type floating, parent Link0, child Link2, origin xyz=-0.009654325011552584 0 3 rpy=0 0 0, axis 0 0 1, limit lower=-3.14159 upper=3.14159 effort=0.0 velocity=0.0
- joint Link0_Link1: origin xyz=0 0 3.7081525025303446 rpy=0 0 0 -> xyz=0 -0.02127435024060903 3 rpy=0 0 0; type continuous -> floating
- joint Link0_Link3: axis 0 1 0 -> 0 0 1; origin xyz=0 -0.6056373343663854 3 rpy=0 0 0 -> xyz=0.009654325011552584 0 3 rpy=0 0 0; type continuous -> revolute

File: samples/sample_3/body3a.urdf (robot description, URDF)
Before this commit: robot robot, 3 links, 2 joints
Links:
- removed link Link3
- added link Link2, mass 1; collision box size=0.4717670957930249 0.39556788109188606 0.4299550821967209; visual box size=0.4717670957930249 0.39556788109188606 0.4299550821967209
- link Link0: geometry collision box size=0.03097385261212171 1.0533102445697646 0.9746180013596537; visual box size=0.03097385261212171 1.0533102445697646 0.9746180013596537
- link Link1: geometry collision box size=0.7465049486349282 1.402582158929547 0.1726767550465887; visual box size=0.7465049486349282 1.402582158929547 0.1726767550465887
Joints:
- removed joint Link0_Link3
- added joint Link0_Link2: type floating, parent Link0, child Link2, origin xyz=0 0.5266551222848823 3 rpy=0 0 0, axis 0 0 1, limit lower=-3.14159 upper=3.14159 effort=0.0 velocity=0.0
- joint Link0_Link1: axis 1 0 0 -> 0 0 1; origin xyz=0 0 3.7081525025303446 rpy=0 0 0 -> xyz=0.015486926306060855 0 3 rpy=0 0 0

File: samples/sample_4/body4a.urdf (robot description, URDF)
Before this commit: robot robot, 3 links, 2 joints
Links:
- link Link0: geometry collision box size=0.6492924829784956 0.6778343287193214 1.0560439675676974; visual box size=0.6492924829784956 0.6778343287193214 1.0560439675676974
- link Link1: geometry collision box size=0.030488788179828696 0.4786016522264719 0.6173334968087147; visual box size=0.030488788179828696 0.4786016522264719 0.6173334968087147
- link Link2: geometry collision box size=1.0155201012278048 1.4909908915539631 1.3578900046341884; visual box size=1.0155201012278048 1.4909908915539631 1.3578900046341884
Joints:
- joint Link0_Link1: origin xyz=0 0 3.7081525025303446 rpy=0 0 0 -> xyz=0 0 3.528021983783849 rpy=0 0 0; type continuous -> floating
- joint Link1_Link2: origin xyz=0.2553621664001794 0 0.6048584974729144 rpy=0 0 0 -> xyz=0 0 0.6173334968087147 rpy=0 0 0; type revolute -> continuous
