Commit message: Finished all sample runs

File: samples/sample_1/body1a.urdf (robot description, URDF)
Before this commit: robot robot, 2 links, 1 joints
Links:
- added link Link2, mass 1; collision box size=0.5961721394320378 1.2292183741672993 0.11109368780118345; visual box size=0.5961721394320378 1.2292183741672993 0.11109368780118345
- link Link0: geometry collision box size=0.5892587456048781 0.9678709277911421 1.102550748417383; visual box size=0.5892587456048781 0.9678709277911421 1.102550748417383
- link Link1: geometry collision box size=0.2387195082361277 0.7979895488258162 1.3206126028535998; visual box size=0.2387195082361277 0.7979895488258162 1.3206126028535998
Joints:
- added joint Link0_Link2: type continuous, parent Link0, child Link2, origin xyz=-0.29462937280243906 0 3 rpy=0 0 0, axis 0 1 0, limit lower=-3.14159 upper=3.14159 effort=0.0 velocity=0.0
- joint Link0_Link1: axis 0 0 1 -> 1 0 0; origin xyz=0 0 3.186444928095009 rpy=0 0 0 -> xyz=0 0 2.4487246257913085 rpy=0 0 0

File: samples/sample_1/body1b.urdf (robot description, URDF)
Before this commit: robot robot, 7 links, 6 joints
Links:
- removed link Link1
- removed link Link4
- removed link Link6
- removed link Link7
- link Link0: geometry collision box size=0.5892587456048781 0.9678709277911421 1.102550748417383; visual box size=0.5892587456048781 0.9678709277911421 1.102550748417383
- link Link2: geometry collision box size=0.5961721394320378 1.2292183741672993 0.11109368780118345; visual box size=0.5961721394320378 1.2292183741672993 0.11109368780118345
- link Link3: geometry collision box size=1.0685510599474437 0.6627356043739749 0.06756053192352834; visual box size=1.0685510599474437 0.6627356043739749 0.06756053192352834
Joints:
- removed joint Link0_Link1
- removed joint Link1_Link2
- removed joint Link3_Link4
- removed joint Link3_Link6
- removed joint Link4_Link7
- added joint Link0_Link2: type continuous, parent Link0, child Link2, origin xyz=-0.29462937280243906 0 3 rpy=0 0 0, axis 0 1 0, limit lower=-3.14159 upper=3.14159 effort=0.0 velocity=0.0
- joint Link2_Link3: origin xyz=-0.22889416297874934 -0.3863325424017958 0 rpy=0 0 0 -> xyz=-0.2980860697160189 0 -0.055546843900591725 rpy=0 0 0

File: samples/sample_1/body1c.urdf (robot description, URDF)
Before this commit: robot robot, 7 links, 6 joints
Links:
- removed link Link1
- removed link Link6
- removed link Link7
- link Link0: geometry collision box size=0.5892587456048781 0.9678709277911421 1.102550748417383; visual box size=0.5892587456048781 0.9678709277911421 1.102550748417383
- link Link2: geometry collision box size=0.5961721394320378 1.2292183741672993 0.11109368780118345; visual box size=0.5961721394320378 1.2292183741672993 0.11109368780118345
- link Link3: geometry collision box size=1.0685510599474437 0.6627356043739749 0.06756053192352834; visual box size=1.0685510599474437 0.6627356043739749 0.06756053192352834
- link Link4: geometry collision box size=1.1908689317751042 1.0738682587664479 0.6939183128569414; visual box size=1.1908689317751042 1.0738682587664479 0.6939183128569414
Joints:
- removed joint Link0_Link1
- removed joint Link1_Link2
- removed joint Link3_Link6
- removed joint Link4_Link7
- added joint Link0_Link2: type continuous, parent Link0, child Link2, origin xyz=-0.29462937280243906 0 3 rpy=0 0 0, axis 0 1 0, limit lower=-3.14159 upper=3.14159 effort=0.0 velocity=0.0
- joint Link2_Link3: origin xyz=-0.22889416297874934 -0.3863325424017958 0 rpy=0 0 0 -> xyz=-0.2980860697160189 0 -0.055546843900591725 rpy=0 0 0
- joint Link3_Link4: axis 1 0 0 -> 0 1 0; origin xyz=0.5845106067746852 -0.6965511835771853 0 rpy=0 0 0 -> xyz=-0.5342755299737219 0 -0.03378026596176417 rpy=0 0 0

File: samples/sample_4/body4b.urdf (robot description, URDF)
Before this commit: robot robot, 7 links, 6 joints
Links:
- removed link Link5
- removed link Link6
- link Link4: geometry collision box size=0.48034767322873323 0.12615857976309708 1.345747834182725; visual box size=0.48034767322873323 0.12615857976309708 1.345747834182725
Joints:
- removed joint Link0_Link5
- removed joint Link0_Link6
- removed joint Link3_Link4
- added joint Link1_Link4: type continuous, parent Link1, child Link4, origin xyz=0 -0.23930082611323594 0.30866674840435737 rpy=0 0 0, axis 1 0 0, limit lower=-3.14159 upper=3.14159 effort=0.0 velocity=0.0

File: samples/sample_4/body4c.urdf (robot description, URDF)
Before this commit: robot robot, 5 links, 4 joints
Links:
- added link Link5, mass 1; collision box size=0.3905442898507795 1.3075422646803185 0.7257314070197918; visual box size=0.3905442898507795 1.3075422646803185 0.7257314070197918
- added link Link6, mass 1; collision box size=0.5399557316528635 0.9085225828426524 0.21272103263793501; visual box size=0.5399557316528635 0.9085225828426524 0.21272103263793501
- link Link4: geometry collision box size=0.6983270117351986 0.6663701868780403 0.19980960062760206; visual box size=0.6983270117351986 0.6663701868780403 0.19980960062760206
Joints:
- removed joint Link1_Link4
- added joint Link0_Link5: type floating, parent Link0, child Link5, origin xyz=0.3246462414892478 0 3 rpy=0 0 0, axis 1 0 0, limit lower=-3.14159 upper=3.14159 effort=0.0 velocity=0.0
- added joint Link0_Link6: type floating, parent Link0, child Link6, origin xyz=0 0.3389171643596607 3 rpy=0 0 0, axis 1 0 0, limit lower=-3.14159 upper=3.14159 effort=0.0 velocity=0.0
- added joint Link3_Link4: type floating, parent Link3, child Link4, origin xyz=0.3659133767641747 0 0.4418005092715366 rpy=0 0 0, axis 0 1 0, limit lower=-3.14159 upper=3.14159 effort=0.0 velocity=0.0
