Commit message: Sample updates

File: samples/sample_3/body3a.urdf (robot description, URDF)
Before this commit: robot robot, 3 links, 2 joints
Links:
- link Link0: geometry collision box size=1.44204024365982 0.2898367197203824 0.17002144968014932; visual box size=1.44204024365982 0.2898367197203824 0.17002144968014932
- link Link1: geometry collision box size=0.11223945369840843 1.1531249653927462 1.281901297000347; visual box size=0.11223945369840843 1.1531249653927462 1.281901297000347
- link Link2: geometry collision box size=0.8279317878985875 1.474640574037379 1.4170488201622882; visual box size=0.8279317878985875 1.474640574037379 1.4170488201622882
Joints:
- joint Link0_Link1: axis 0 0 1 -> 1 0 0; origin xyz=0.015486926306060855 0 3 rpy=0 0 0 -> xyz=0 0.1449183598601912 3 rpy=0 0 0; type continuous -> revolute
- joint Link0_Link2: axis 0 0 1 -> 0 1 0; origin xyz=0 0.5266551222848823 3 rpy=0 0 0 -> xyz=0.72102012182991 0 3 rpy=0 0 0; type floating -> revolute

File: samples/sample_3/body3b.urdf (robot description, URDF)
Before this commit: robot robot, 5 links, 4 joints
Links:
- removed link Link6
- removed link Link7
- added link Link2, mass 1; collision box size=0.8279317878985875 1.474640574037379 1.4170488201622882; visual box size=0.8279317878985875 1.474640574037379 1.4170488201622882
- link Link0: geometry collision box size=1.44204024365982 0.2898367197203824 0.17002144968014932; visual box size=1.44204024365982 0.2898367197203824 0.17002144968014932
- link Link3: geometry collision box size=0.9715027287766891 0.22034239248865067 0.8413341868631763; visual box size=0.9715027287766891 0.22034239248865067 0.8413341868631763
- link Link4: geometry collision box size=0.5177231618015214 0.21320700012698124 1.3186578187042433; visual box size=0.5177231618015214 0.21320700012698124 1.3186578187042433
Joints:
- removed joint Link0_Link3
- removed joint Link3_Link4
- removed joint Link4_Link6
- removed joint Link4_Link7
- added joint Link0_Link2: type revolute, parent Link0, child Link2, origin xyz=0.72102012182991 0 3 rpy=0 0 0, axis 0 1 0, limit lower=-3.14159 upper=3.14159 effort=0.0 velocity=0.0
- added joint Link0_Link4: type continuous, parent Link0, child Link4, origin xyz=0 0 3.0850107248400747 rpy=0 0 0, axis 0 1 0, limit lower=-3.14159 upper=3.14159 effort=0.0 velocity=0.0
- added joint Link2_Link3: type revolute, parent Link2, child Link3, origin xyz=0.41396589394929373 0 -0.7085244100811441 rpy=0 0 0, axis 0 1 0, limit lower=-3.14159 upper=3.14159 effort=0.0 velocity=0.0

File: samples/sample_3/body3c.urdf (robot description, URDF)
Before this commit: robot robot, 7 links, 6 joints
Links:
- removed link Link6
- removed link Link7
- removed link Link8
- added link Link2, mass 1; collision box size=0.8279317878985875 1.474640574037379 1.4170488201622882; visual box size=0.8279317878985875 1.474640574037379 1.4170488201622882
- link Link0: geometry collision box size=1.44204024365982 0.2898367197203824 0.17002144968014932; visual box size=1.44204024365982 0.2898367197203824 0.17002144968014932
- link Link3: geometry collision box size=0.9715027287766891 0.22034239248865067 0.8413341868631763; visual box size=0.9715027287766891 0.22034239248865067 0.8413341868631763
- link Link4: geometry collision box size=0.5177231618015214 0.21320700012698124 1.3186578187042433; visual box size=0.5177231618015214 0.21320700012698124 1.3186578187042433
- link Link5: geometry collision box size=0.32366369255784205 0.5237724945873385 1.3343994731736073; visual box size=0.32366369255784205 0.5237724945873385 1.3343994731736073
Joints:
- removed joint Link0_Link3
- removed joint Link0_Link8
- removed joint Link3_Link4
- removed joint Link4_Link6
- removed joint Link4_Link7
- added joint Link0_Link2: type revolute, parent Link0, child Link2, origin xyz=0.72102012182991 0 3 rpy=0 0 0, axis 0 1 0, limit lower=-3.14159 upper=3.14159 effort=0.0 velocity=0.0
- added joint Link0_Link4: type continuous, parent Link0, child Link4, origin xyz=0 0 3.0850107248400747 rpy=0 0 0, axis 0 1 0, limit lower=-3.14159 upper=3.14159 effort=0.0 velocity=0.0
- added joint Link2_Link3: type revolute, parent Link2, child Link3, origin xyz=0.41396589394929373 0 -0.7085244100811441 rpy=0 0 0, axis 0 1 0, limit lower=-3.14159 upper=3.14159 effort=0.0 velocity=0.0
- joint Link3_Link5: axis 0 0 1 -> 0 1 0; origin xyz=0 0.3121865513005121 -0.4160462490743261 rpy=0 0 0 -> xyz=-0.48575136438834454 0 -0.42066709343158815 rpy=0 0 0

File: samples/sample_5/body5a.urdf (robot description, URDF)
Before this commit: robot robot, 2 links, 1 joints
Links:
- link Link0: geometry collision box size=0.8295870886287884 1.3089110557684878 1.2975801466922856; visual box size=0.8295870886287884 1.3089110557684878 1.2975801466922856
- link Link1: geometry collision box size=0.7905171132797519 0.7066909116991853 0.9591370686578011; visual box size=0.7905171132797519 0.7066909116991853 0.9591370686578011
Joints:
- joint Link0_Link1: axis 1 0 0 -> 0 1 0; origin xyz=0.4907325711572144 0 3 rpy=0 0 0 -> xyz=0 0 3.648790073346143 rpy=0 0 0; type continuous -> revolute

File: samples/sample_5/body5b.urdf (robot description, URDF)
Before this commit: robot robot, 6 links, 5 joints
Links:
- removed link Link4
- removed link Link6
- removed link Link7
- added link Link1, mass 1; collision box size=0.7905171132797519 0.7066909116991853 0.9591370686578011; visual box size=0.7905171132797519 0.7066909116991853 0.9591370686578011
- link Link0: geometry collision box size=0.8295870886287884 1.3089110557684878 1.2975801466922856; visual box size=0.8295870886287884 1.3089110557684878 1.2975801466922856
- link Link2: geometry collision box size=0.7394819814481246 1.0378329166671527 0.5236035340144687; visual box size=0.7394819814481246 1.0378329166671527 0.5236035340144687
- link Link3: geometry collision box size=0.7991792016202215 0.4897041070484848 1.200176138982795; visual box size=0.7991792016202215 0.4897041070484848 1.200176138982795
Joints:
- removed joint Link0_Link2
- removed joint Link2_Link3
- removed joint Link3_Link4
- removed joint Link4_Link6
- removed joint Link4_Link7
- added joint Link0_Link1: type revolute, parent Link0, child Link1, origin xyz=0 0 3.648790073346143 rpy=0 0 0, axis 0 1 0, limit lower=-3.14159 upper=3.14159 effort=0.0 velocity=0.0
- added joint Link1_Link2: type revolute, parent Link1, child Link2, origin xyz=0.39525855663987597 0 0.47956853432890056 rpy=0 0 0, axis 0 1 0, limit lower=-3.14159 upper=3.14159 effort=0.0 velocity=0.0
- added joint Link1_Link3: type floating, parent Link1, child Link3, origin xyz=0 -0.35334545584959265 0.47956853432890056 rpy=0 0 0, axis 0 0 1, limit lower=-3.14159 upper=3.14159 effort=0.0 velocity=0.0

File: samples/sample_5/body5c.urdf (robot description, URDF)
Before this commit: robot robot, 7 links, 6 joints
Links:
- removed link Link3
- removed link Link4
- removed link Link6
- removed link Link7
- link Link0: geometry collision box size=0.8295870886287884 1.3089110557684878 1.2975801466922856; visual box size=0.8295870886287884 1.3089110557684878 1.2975801466922856
- link Link1: geometry collision box size=0.7905171132797519 0.7066909116991853 0.9591370686578011; visual box size=0.7905171132797519 0.7066909116991853 0.9591370686578011
- link Link2: geometry collision box size=0.7394819814481246 1.0378329166671527 0.5236035340144687; visual box size=0.7394819814481246 1.0378329166671527 0.5236035340144687
Joints:
- removed joint Link0_Link2
- removed joint Link2_Link3
- removed joint Link3_Link4
- removed joint Link4_Link6
- removed joint Link4_Link7
- added joint Link1_Link2: type revolute, parent Link1, child Link2, origin xyz=0.39525855663987597 0 0.47956853432890056 rpy=0 0 0, axis 0 1 0, limit lower=-3.14159 upper=3.14159 effort=0.0 velocity=0.0
- joint Link0_Link1: axis 1 0 0 -> 0 1 0; origin xyz=0.4907325711572144 0 3 rpy=0 0 0 -> xyz=0 0 3.648790073346143 rpy=0 0 0; type continuous -> revolute

File: samples/sample_6/body6a.urdf (robot description, URDF)
Before this commit: robot robot, 2 links, 1 joints
Links:
- added link Link2, mass 1; collision box size=0.4717670957930249 0.39556788109188606 0.4299550821967209; visual box size=0.4717670957930249 0.39556788109188606 0.4299550821967209
- link Link0: geometry collision box size=0.03097385261212171 1.0533102445697646 0.9746180013596537; visual box size=0.03097385261212171 1.0533102445697646 0.9746180013596537
- link Link1: geometry collision box size=0.7465049486349282 1.402582158929547 0.1726767550465887; visual box size=0.7465049486349282 1.402582158929547 0.1726767550465887
Joints:
- added joint Link0_Link2: type floating, parent Link0, child Link2, origin xyz=0 0.5266551222848823 3 rpy=0 0 0, axis 0 0 1, limit lower=-3.14159 upper=3.14159 effort=0.0 velocity=0.0
- joint Link0_Link1: axis 0 1 0 -> 0 0 1; origin xyz=0 0 3.648790073346143 rpy=0 0 0 -> xyz=0.015486926306060855 0 3 rpy=0 0 0; type revolute -> continuous

File: samples/sample_6/body6b.urdf (robot description, URDF)
Before this commit: robot robot, 4 links, 3 joints
Links:
- removed link Link1
- removed link Link2
- added link Link4, mass 1; collision box size=0.19393852368441028 0.5566570656606415 0.5996958965262241; visual box size=0.19393852368441028 0.5566570656606415 0.5996958965262241
- added link Link6, mass 1; collision box size=0.07606633735372897 0.03652848300226824 0.8881153104232047; visual box size=0.07606633735372897 0.03652848300226824 0.8881153104232047
- added link Link7, mass 1; collision box size=0.8720057671767885 1.1240179037474778 1.1004631064480914; visual box size=0.8720057671767885 1.1240179037474778 1.1004631064480914
- link Link0: geometry collision box size=0.03097385261212171 1.0533102445697646 0.9746180013596537; visual box size=0.03097385261212171 1.0533102445697646 0.9746180013596537
- link Link3: geometry collision box size=0.9748677807526844 0.6243731026010242 0.8320924981486522; visual box size=0.9748677807526844 0.6243731026010242 0.8320924981486522
Joints:
- removed joint Link0_Link1
- removed joint Link1_Link2
- removed joint Link1_Link3
- added joint Link0_Link3: type floating, parent Link0, child Link3, origin xyz=0 0 2.5126909993201734 rpy=0 0 0, axis 0 0 1, limit lower=-3.14159 upper=3.14159 effort=0.0 velocity=0.0
- added joint Link3_Link4: type revolute, parent Link3, child Link4, origin xyz=0 -0.3121865513005121 -0.4160462490743261 rpy=0 0 0, axis 0 0 1, limit lower=-3.14159 upper=3.14159 effort=0.0 velocity=0.0
- added joint Link4_Link6: type continuous, parent Link4, child Link6, origin xyz=0 -0.5566570656606415 0 rpy=0 0 0, axis 0 0 1, limit lower=-3.14159 upper=3.14159 effort=0.0 velocity=0.0
- added joint Link4_Link7: type revolute, parent Link4, child Link7, origin xyz=-0.09696926184220514 -0.2783285328303208 0 rpy=0 0 0, axis 1 0 0, limit lower=-3.14159 upper=3.14159 effort=0.0 velocity=0.0

File: samples/sample_6/body6c.urdf (robot description, URDF)
Before this commit: robot robot, 3 links, 2 joints
Links:
- removed link Link1
- removed link Link2
- added link Link3, mass 1; collision box size=0.9748677807526844 0.6243731026010242 0.8320924981486522; visual box size=0.9748677807526844 0.6243731026010242 0.8320924981486522
- added link Link4, mass 1; collision box size=0.19393852368441028 0.5566570656606415 0.5996958965262241; visual box size=0.19393852368441028 0.5566570656606415 0.5996958965262241
- added link Link5, mass 1; collision box size=1.0631376200435807 1.3704597332400164 0.3775299092337461; visual box size=1.0631376200435807 1.3704597332400164 0.3775299092337461
- added link Link6, mass 1; collision box size=0.07606633735372897 0.03652848300226824 0.8881153104232047; visual box size=0.07606633735372897 0.03652848300226824 0.8881153104232047
- added link Link7, mass 1; collision box size=0.8720057671767885 1.1240179037474778 1.1004631064480914; visual box size=0.8720057671767885 1.1240179037474778 1.1004631064480914
- added link Link8, mass 1; collision box size=1.4757175967173934 0.8485635371437219 1.371338483094021; visual box size=1.4757175967173934 0.8485635371437219 1.371338483094021
- link Link0: geometry collision box size=0.03097385261212171 1.0533102445697646 0.9746180013596537; visual box size=0.03097385261212171 1.0533102445697646 0.9746180013596537
Joints:
- removed joint Link0_Link1
- removed joint Link1_Link2
- added joint Link0_Link3: type floating, parent Link0, child Link3, origin xyz=0 0 2.5126909993201734 rpy=0 0 0, axis 0 0 1, limit lower=-3.14159 upper=3.14159 effort=0.0 velocity=0.0
- added joint Link0_Link8: type floating, parent Link0, child Link8, origin xyz=-0.015486926306060855 0 3 rpy=0 0 0, axis 0 1 0, limit lower=-3.14159 upper=3.14159 effort=0.0 velocity=0.0
- added joint Link3_Link4: type revolute, parent Link3, child Link4, origin xyz=0 -0.3121865513005121 -0.4160462490743261 rpy=0 0 0, axis 0 0 1, limit lower=-3.14159 upper=3.14159 effort=0.0 velocity=0.0
- added joint Link3_Link5: type floating, parent Link3, child Link5, origin xyz=0 0.3121865513005121 -0.4160462490743261 rpy=0 0 0, axis 0 0 1, limit lower=-3.14159 upper=3.14159 effort=0.0 velocity=0.0
- added joint Link4_Link6: type continuous, parent Link4, child Link6, origin xyz=0 -0.5566570656606415 0 rpy=0 0 0, axis 0 0 1, limit lower=-3.14159 upper=3.14159 effort=0.0 velocity=0.0
- added joint Link4_Link7: type revolute, parent Link4, child Link7, origin xyz=-0.09696926184220514 -0.2783285328303208 0 rpy=0 0 0, axis 1 0 0, limit lower=-3.14159 upper=3.14159 effort=0.0 velocity=0.0

File: samples/sample_9/body9a.urdf (robot description, URDF)
Before this commit: robot robot, 3 links, 2 joints
Links:
- removed link Link2
- link Link0: geometry collision box size=0.9814651423144288 0.9724103184434222 1.2869403903583185; visual box size=0.9814651423144288 0.9724103184434222 1.2869403903583185
- link Link1: geometry collision box size=1.0018625360092275 0.3238134013247041 0.08046545417389306; visual box size=1.0018625360092275 0.3238134013247041 0.08046545417389306
Joints:
- removed joint Link0_Link2
- joint Link0_Link1: origin xyz=0 0.1449183598601912 3 rpy=0 0 0 -> xyz=0.4907325711572144 0 3 rpy=0 0 0; type revolute -> continuous

File: samples/sample_9/body9b.urdf (robot description, URDF)
Before this commit: robot robot, 4 links, 3 joints
Links:
- added link Link6, mass 1; collision box size=0.12666363385725105 1.2977454902383796 0.023724270103385403; visual box size=0.12666363385725105 1.2977454902383796 0.023724270103385403
- added link Link7, mass 1; collision box size=0.12543833849260377 0.8630309022970761 0.8503725666685922; visual box size=0.12543833849260377 0.8630309022970761 0.8503725666685922
- link Link0: geometry collision box size=0.9814651423144288 0.9724103184434222 1.2869403903583185; visual box size=0.9814651423144288 0.9724103184434222 1.2869403903583185
- link Link2: geometry collision box size=1.1675008126636683 1.2992007133460834 1.0787933767438094; visual box size=1.1675008126636683 1.2992007133460834 1.0787933767438094
- link Link3: geometry collision box size=0.02854000632289 1.4153058076502172 0.6797410429779047; visual box size=0.02854000632289 1.4153058076502172 0.6797410429779047
- link Link4: geometry collision box size=0.7452616532996463 1.3811815948738264 0.9536310773481043; visual box size=0.7452616532996463 1.3811815948738264 0.9536310773481043
Joints:
- removed joint Link0_Link4
- added joint Link3_Link4: type revolute, parent Link3, child Link4, origin xyz=-0.02854000632289 0 0 rpy=0 0 0, axis 1 0 0, limit lower=-3.14159 upper=3.14159 effort=0.0 velocity=0.0
- added joint Link4_Link6: type continuous, parent Link4, child Link6, origin xyz=-0.37263082664982317 0 0.47681553867405213 rpy=0 0 0, axis 0 0 1, limit lower=-3.14159 upper=3.14159 effort=0.0 velocity=0.0
- added joint Link4_Link7: type revolute, parent Link4, child Link7, origin xyz=-0.37263082664982317 0.6905907974369132 0 rpy=0 0 0, axis 0 0 1, limit lower=-3.14159 upper=3.14159 effort=0.0 velocity=0.0
- joint Link0_Link2: axis 0 1 0 -> 1 0 0; origin xyz=0.72102012182991 0 3 rpy=0 0 0 -> xyz=-0.4907325711572144 0 3 rpy=0 0 0
- joint Link2_Link3: axis 0 1 0 -> 1 0 0; origin xyz=0.41396589394929373 0 -0.7085244100811441 rpy=0 0 0 -> xyz=-1.1675008126636683 0 0 rpy=0 0 0

File: samples/sample_9/body9c.urdf (robot description, URDF)
Before this commit: robot robot, 5 links, 4 joints
Links:
- removed link Link5
- added link Link1, mass 1; collision box size=1.0018625360092275 0.3238134013247041 0.08046545417389306; visual box size=1.0018625360092275 0.3238134013247041 0.08046545417389306
- added link Link6, mass 1; collision box size=0.12666363385725105 1.2977454902383796 0.023724270103385403; visual box size=0.12666363385725105 1.2977454902383796 0.023724270103385403
- added link Link7, mass 1; collision box size=0.12543833849260377 0.8630309022970761 0.8503725666685922; visual box size=0.12543833849260377 0.8630309022970761 0.8503725666685922
- link Link0: geometry collision box size=0.9814651423144288 0.9724103184434222 1.2869403903583185; visual box size=0.9814651423144288 0.9724103184434222 1.2869403903583185
- link Link2: geometry collision box size=1.1675008126636683 1.2992007133460834 1.0787933767438094; visual box size=1.1675008126636683 1.2992007133460834 1.0787933767438094
- link Link3: geometry collision box size=0.02854000632289 1.4153058076502172 0.6797410429779047; visual box size=0.02854000632289 1.4153058076502172 0.6797410429779047
- link Link4: geometry collision box size=0.7452616532996463 1.3811815948738264 0.9536310773481043; visual box size=0.7452616532996463 1.3811815948738264 0.9536310773481043
Joints:
- removed joint Link0_Link4
- removed joint Link3_Link5
- added joint Link0_Link1: type continuous, parent Link0, child Link1, origin xyz=0.4907325711572144 0 3 rpy=0 0 0, axis 1 0 0, limit lower=-3.14159 upper=3.14159 effort=0.0 velocity=0.0
- added joint Link3_Link4: type revolute, parent Link3, child Link4, origin xyz=-0.02854000632289 0 0 rpy=0 0 0, axis 1 0 0, limit lower=-3.14159 upper=3.14159 effort=0.0 velocity=0.0
- added joint Link4_Link6: type continuous, parent Link4, child Link6, origin xyz=-0.37263082664982317 0 0.47681553867405213 rpy=0 0 0, axis 0 0 1, limit lower=-3.14159 upper=3.14159 effort=0.0 velocity=0.0
- added joint Link4_Link7: type revolute, parent Link4, child Link7, origin xyz=-0.37263082664982317 0.6905907974369132 0 rpy=0 0 0, axis 0 0 1, limit lower=-3.14159 upper=3.14159 effort=0.0 velocity=0.0
- joint Link0_Link2: axis 0 1 0 -> 1 0 0; origin xyz=0.72102012182991 0 3 rpy=0 0 0 -> xyz=-0.4907325711572144 0 3 rpy=0 0 0
- joint Link2_Link3: axis 0 1 0 -> 1 0 0; origin xyz=0.41396589394929373 0 -0.7085244100811441 rpy=0 0 0 -> xyz=-1.1675008126636683 0 0 rpy=0 0 0
